Commit message: setup changes for (hopefully) final static case results

File: conveyor_belt_tamp/models/boxes/black_box.urdf (robot description, URDF)
Before this commit: robot black_box, 1 links, 0 joints
Links:
- link base_link: geometry collision box size=0.059 0.059 0.149; collision sphere radius=1e-7

File: conveyor_belt_tamp/models/boxes/black_box10.urdf (robot description, URDF)
Before this commit: robot black_box10, 1 links, 0 joints
Links:
- link base_link: mass 0.1 -> 0.122; geometry collision box size=0.064 0.054 0.149; collision sphere radius=1e-7

File: conveyor_belt_tamp/models/boxes/black_box11.urdf (robot description, URDF)
Before this commit: robot black_box11, 1 links, 0 joints
Links:
- link base_link: mass 0.1 -> 0.122; geometry collision box size=0.064 0.054 0.149; collision sphere radius=1e-7

File: conveyor_belt_tamp/models/boxes/black_box12.urdf (robot description, URDF)
Before this commit: robot black_box12, 1 links, 0 joints
Links:
- link base_link: mass 0.1 -> 0.122; geometry collision box size=0.064 0.054 0.149; collision sphere radius=1e-7

File: conveyor_belt_tamp/models/boxes/black_box2.urdf (robot description, URDF)
Before this commit: robot black_box2, 1 links, 0 joints
Links:
- link base_link: geometry collision box size=0.064 0.054 0.149; collision sphere radius=1e-7

File: conveyor_belt_tamp/models/boxes/black_box3.urdf (robot description, URDF)
Before this commit: robot black_box3, 1 links, 0 joints
Links:
- link base_link: geometry collision box size=0.064 0.054 0.149; collision sphere radius=1e-7

File: conveyor_belt_tamp/models/boxes/black_box4.urdf (robot description, URDF)
Before this commit: robot black_box4, 1 links, 0 joints
Links:
- link base_link: geometry collision box size=0.064 0.054 0.149; collision sphere radius=1e-7

File: conveyor_belt_tamp/models/boxes/black_box5.urdf (robot description, URDF)
Before this commit: robot black_box5, 1 links, 0 joints
Links:
- link base_link: mass 0.1 -> 0.122; geometry collision box size=0.064 0.054 0.149; collision sphere radius=1e-7

File: conveyor_belt_tamp/models/boxes/black_box6.urdf (robot description, URDF)
Before this commit: robot black_box6, 1 links, 0 joints
Links:
- link base_link: mass 0.1 -> 0.122; geometry collision box size=0.064 0.054 0.149; collision sphere radius=1e-7

File: conveyor_belt_tamp/models/boxes/black_box7.urdf (robot description, URDF)
Before this commit: robot black_box7, 1 links, 0 joints
Links:
- link base_link: mass 0.1 -> 0.122; geometry collision box size=0.064 0.054 0.149; collision sphere radius=1e-7

File: conveyor_belt_tamp/models/boxes/black_box8.urdf (robot description, URDF)
Before this commit: robot black_box8, 1 links, 0 joints
Links:
- link base_link: mass 0.1 -> 0.122; geometry collision box size=0.064 0.054 0.149; collision sphere radius=1e-7

File: conveyor_belt_tamp/models/boxes/black_box9.urdf (robot description, URDF)
Before this commit: robot black_box9, 1 links, 0 joints
Links:
- link base_link: mass 0.1 -> 0.122; geometry collision box size=0.064 0.054 0.149; collision sphere radius=1e-7

File: conveyor_belt_tamp/models/boxes/redblock.urdf (robot description, URDF)
Before this commit: robot simple_cuboid, 1 links, 0 joints
Links:
- link base_link: geometry collision box size=0.059 0.059 0.149; collision sphere radius=1e-7

File: conveyor_belt_tamp/models/boxes/redblock2.urdf (robot description, URDF)
Before this commit: robot simple_cuboid2, 1 links, 0 joints
Links:
- link base_link: geometry collision box size=0.059 0.059 0.149; collision sphere radius=1e-7

Commit message: conveyor belt scenario modifications

File: conveyor_belt_tamp/models/boxes/black_box.urdf (robot description, URDF)
Before this commit: robot black_box, 1 links, 0 joints
Links:
- link base_link: mass 0.1 -> 0.122; geometry collision box size=0.064 0.054 0.169; collision sphere radius=1e-7

File: conveyor_belt_tamp/models/boxes/black_box10.urdf (robot description, URDF)
Before this commit: robot black_box10, 1 links, 0 joints
Links:
- link base_link: geometry collision box size=0.064 0.054 0.169; collision sphere radius=1e-7

File: conveyor_belt_tamp/models/boxes/black_box11.urdf (robot description, URDF)
Before this commit: robot black_box11, 1 links, 0 joints
Links:
- link base_link: geometry collision box size=0.064 0.054 0.169; collision sphere radius=1e-7

File: conveyor_belt_tamp/models/boxes/black_box12.urdf (robot description, URDF)
Before this commit: robot black_box12, 1 links, 0 joints
Links:
- link base_link: geometry collision box size=0.064 0.054 0.169; collision sphere radius=1e-7

File: conveyor_belt_tamp/models/boxes/black_box2.urdf (robot description, URDF)
Before this commit: robot black_box2, 1 links, 0 joints
Links:
- link base_link: geometry collision box size=0.064 0.054 0.169; collision sphere radius=1e-7

File: conveyor_belt_tamp/models/boxes/black_box3.urdf (robot description, URDF)
Before this commit: robot black_box3, 1 links, 0 joints
Links:
- link base_link: geometry collision box size=0.064 0.054 0.169; collision sphere radius=1e-7

File: conveyor_belt_tamp/models/boxes/black_box4.urdf (robot description, URDF)
Before this commit: robot black_box4, 1 links, 0 joints
Links:
- link base_link: geometry collision box size=0.064 0.054 0.169; collision sphere radius=1e-7

File: conveyor_belt_tamp/models/boxes/black_box5.urdf (robot description, URDF)
Before this commit: robot black_box5, 1 links, 0 joints
Links:
- link base_link: geometry collision box size=0.064 0.054 0.169; collision sphere radius=1e-7

File: conveyor_belt_tamp/models/boxes/black_box6.urdf (robot description, URDF)
Before this commit: robot black_box6, 1 links, 0 joints
Links:
- link base_link: geometry collision box size=0.064 0.054 0.169; collision sphere radius=1e-7

File: conveyor_belt_tamp/models/boxes/black_box7.urdf (robot description, URDF)
Before this commit: robot black_box7, 1 links, 0 joints
Links:
- link base_link: geometry collision box size=0.064 0.054 0.169; collision sphere radius=1e-7

File: conveyor_belt_tamp/models/boxes/black_box8.urdf (robot description, URDF)
Before this commit: robot black_box8, 1 links, 0 joints
Links:
- link base_link: geometry collision box size=0.064 0.054 0.169; collision sphere radius=1e-7

File: conveyor_belt_tamp/models/boxes/black_box9.urdf (robot description, URDF)
Before this commit: robot black_box9, 1 links, 0 joints
Links:
- link base_link: geometry collision box size=0.064 0.054 0.169; collision sphere radius=1e-7

File: conveyor_belt_tamp/models/boxes/redblock.urdf (robot description, URDF)
Before this commit: robot simple_cuboid, 1 links, 0 joints
Links:
- link base_link: geometry collision box size=0.059 0.059 0.169; collision sphere radius=1e-7

File: conveyor_belt_tamp/models/boxes/redblock2.urdf (robot description, URDF)
Before this commit: robot simple_cuboid2, 1 links, 0 joints
Links:
- link base_link: geometry collision box size=0.059 0.059 0.169; collision sphere radius=1e-7
